File: FY6600_Power_Supply.sch (KiCad schematic (older format))
At the start: 57 parts, among them J1 Conn_01x02, J2 Conn_01x06, J3 Conn_01x02, SW1 SW_SPST, T1 Transformer_1P_1S, T2 Transformer_1P_2S, U1 LM7805_TO220, U2 LM317_TO-220, U3 LM337_TO220

Commit message: Interactive BOM
Parts:
- C1, C5, C9: value 2200u -> 4700u
- R2, R6: value 8.2k -> 6.8k
- R3: value 2.2k -> 3.3k
- R4, R5: value 4.7k -> 10k
- RV1, RV2: value 3.3k -> 4.7k
Other:
- note added: "Vout = 1.25V * (1 + (R2+RV1)/R1)\nVmin = 1.25V * (1 + 6.8k/1k) = 9.75V\nVmax = 1.25V * (1 + 11.5k/1k) = 15.6V"
- note removed: "Vout = 1.25V * (1 + (R2+RV1)/R1)\nVmin = 1.25V * (1 + 8.2k/1k) = 11.5V\nVmax = 1.25V * (1 + 11.5k/1k) = 15.6V"
Changed lines of the file:
@@
 P 5050 1600
 F 0 "C1" H 5138 1646 50  0000 L CNN
-F 1 "2200u" H 5138 1555 50  0000 L CNN
+F 1 "4700u" H 5138 1555 50  0000 L CNN
 F 2 "Capacitor_THT:CP_Radial_D18.0mm_P7.50mm" H 5050 1600 50  0001 C CNN
 F 3 "~" H 5050 1600 50  0001 C CNN
@@
 P 5050 3700
 F 0 "C5" H 5138 3746 50  0000 L CNN
-F 1 "2200u" H 5138 3655 50  0000 L CNN
+F 1 "4700u" H 5138 3655 50  0000 L CNN
 F 2 "Capacitor_THT:CP_Radial_D18.0mm_P7.50mm" H 5050 3700 50  0001 C CNN
 F 3 "~" H 5050 3700 50  0001 C CNN
@@
 P 5050 5100
 F 0 "C9" H 5138 5146 50  0000 L CNN
-F 1 "2200u" H 5138 5055 50  0000 L CNN
+F 1 "4700u" H 5138 5055 50  0000 L CNN
 F 2 "Capacitor_THT:CP_Radial_D18.0mm_P7.50mm" H 5050 5100 50  0001 C CNN
 F 3 "~" H 5050 5100 50  0001 C CNN
@@
 P 5800 3900
 F 0 "R2" H 5870 3946 50  0000 L CNN
-F 1 "8.2k" H 5870 3855 50  0000 L CNN
+F 1 "6.8k" H 5870 3855 50  0000 L CNN
 F 2 "Resistor_SMD:R_0805_2012Metric_Pad1.20x1.40mm_HandSolder" V 5730 3900 50  0001 C CNN
 F 3 "~" H 5800 3900 50  0001 C CNN
@@
 P 5800 4200
 F 0 "RV1" H 5730 4246 50  0000 R CNN
-F 1 "3.3k" H 5730 4155 50  0000 R CNN
+F 1 "4.7k" H 5730 4155 50  0000 R CNN
 F 2 "Potentiometer_THT:Potentiometer_Piher_PT-6-V_Vertical" H 5800 4200 50  0001 C CNN
 F 3 "~" H 5800 4200 50  0001 C CNN
@@
 P 5800 4900
 F 0 "R6" H 5870 4946 50  0000 L CNN
-F 1 "8.2k" H 5870 4855 50  0000 L CNN
+F 1 "6.8k" H 5870 4855 50  0000 L CNN
 F 2 "Resistor_SMD:R_0805_2012Metric_Pad1.20x1.40mm_HandSolder" V 5730 4900 50  0001 C CNN
 F 3 "~" H 5800 4900 50  0001 C CNN
@@
 P 5800 4600
 F 0 "RV2" H 5730 4646 50  0000 R CNN
-F 1 "3.3k" H 5730 4555 50  0000 R CNN
+F 1 "4.7k" H 5730 4555 50  0000 R CNN
 F 2 "Potentiometer_THT:Potentiometer_Piher_PT-6-V_Vertical" H 5800 4600 50  0001 C CNN
 F 3 "~" H 5800 4600 50  0001 C CNN
@@
 	5450 3350 5050 3350
 Text Notes 3650 3150 0    50   ~ 0
-Vout = 1.25V * (1 + (R2+RV1)/R1)\nVmin = 1.25V * (1 + 8.2k/1k) = 11.5V\nVmax = 1.25V * (1 + 11.5k/1k) = 15.6V
+Vout = 1.25V * (1 + (R2+RV1)/R1)\nVmin = 1.25V * (1 + 6.8k/1k) = 9.75V\nVmax = 1.25V * (1 + 11.5k/1k) = 15.6V
 $Comp
 L Device:C_Small C2
@@
 P 9450 3800
 F 0 "R3" H 9520 3846 50  0000 L CNN
-F 1 "2.2k" H 9520 3755 50  0000 L CNN
+F 1 "3.3k" H 9520 3755 50  0000 L CNN
 F 2 "Resistor_SMD:R_0805_2012Metric_Pad1.20x1.40mm_HandSolder" V 9380 3800 50  0001 C CNN
 F 3 "~" H 9450 3800 50  0001 C CNN
@@
 P 9750 3800
 F 0 "R4" H 9820 3846 50  0000 L CNN
-F 1 "4.7k" H 9820 3755 50  0000 L CNN
+F 1 "10k" H 9820 3755 50  0000 L CNN
 F 2 "Resistor_SMD:R_0805_2012Metric_Pad1.20x1.40mm_HandSolder" V 9680 3800 50  0001 C CNN
 F 3 "~" H 9750 3800 50  0001 C CNN
@@
 P 10050 3800
 F 0 "R5" H 10120 3846 50  0000 L CNN
-F 1 "4.7k" H 10120 3755 50  0000 L CNN
+F 1 "10k" H 10120 3755 50  0000 L CNN
 F 2 "Resistor_SMD:R_0805_2012Metric_Pad1.20x1.40mm_HandSolder" V 9980 3800 50  0001 C CNN
 F 3 "~" H 10050 3800 50  0001 C CNN
