File: FY6600_Power_Supply.kicad_pcb (KiCad board)
At the start: 2 copper layers, 95 x 100 mm, 58 parts, among them J1 Conn_01x02, J2 Conn_01x06, J3 Conn_01x02, SW1 SW_SPST, T1 Transformer_1P_1S, T2 Transformer_1P_2S, U1 LM7805_TO220, U2 LM317_TO-220, U3 LM337_TO220

Commit message: Interactive BOM
Parts:
- R2, R6: value 8.2k -> 6.8k
- R3: value 2.2k -> 3.3k
- R4, R5: value 4.7k -> 10k
- RV1, RV2: value 3.3k -> 4.7k
Changed lines of the file:
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@@
       (effects (font (size 1 1) (thickness 0.15)))
     )
-    (fp_text value 3.3k (at 2.5 2.06) (layer F.Fab)
+    (fp_text value 4.7k (at 2.5 2.06) (layer F.Fab)
       (effects (font (size 1 1) (thickness 0.15)))
     )
@@
       (effects (font (size 1 1) (thickness 0.15)))
     )
-    (fp_text value 3.3k (at 2.5 2.06) (layer F.Fab)
+    (fp_text value 4.7k (at 2.5 2.06) (layer F.Fab)
       (effects (font (size 1 1) (thickness 0.15)))
     )
@@
       (effects (font (size 1 1) (thickness 0.15)))
     )
-    (fp_text value 8.2k (at 0 1.65 90) (layer F.Fab)
+    (fp_text value 6.8k (at 0 1.65 90) (layer F.Fab)
       (effects (font (size 1 1) (thickness 0.15)))
     )
@@
       (effects (font (size 1 1) (thickness 0.15)))
     )
-    (fp_text value 4.7k (at 0 1.65 90) (layer F.Fab)
+    (fp_text value 10k (at 0 1.65 90) (layer F.Fab)
       (effects (font (size 1 1) (thickness 0.15)))
     )
@@
       (effects (font (size 1 1) (thickness 0.15)))
     )
-    (fp_text value 4.7k (at 0 1.65 90) (layer F.Fab)
+    (fp_text value 10k (at 0 1.65 90) (layer F.Fab)
       (effects (font (size 1 1) (thickness 0.15)))
     )
@@
       (effects (font (size 1 1) (thickness 0.15)))
     )
-    (fp_text value 2.2k (at 0 1.65 90) (layer F.Fab)
+    (fp_text value 3.3k (at 0 1.65 90) (layer F.Fab)
       (effects (font (size 1 1) (thickness 0.15)))
     )
@@
       (effects (font (size 1 1) (thickness 0.15)))
     )
-    (fp_text value 8.2k (at 0 1.65 90) (layer F.Fab)
-      (effects (font (size 1 1) (thickness 0.15)))
-    )
+    (fp_text value 6.8k (at 0 1.65 90) (layer F.Fab)
+      (effects (font (size 1 1) (thickness 0.15)))
+    )
